File: faden/kicad/faden/faden.kicad_pcb (KiCad board)
At the start: 2 copper layers, 34 parts, among them J1Power1 Conn_01x02_Male, J2Signal1 Conn_01x04_Male, SW1 SW_DPDT_x2, U1 TL082

Commit message: final layout for strip layout
Parts:
- added D8: DIODE, Diode_THT:D_DO-15_P10.16mm_Horizontal, F.Cu at (76.2, 50.8)
- moved RV2 117.3 mm to (76.2, 81.3)
- moved D1 96.7 mm to (96.5, 81.3)
- moved RV1 94.3 mm to (76.2, 86.4)
- moved R6 94.3 mm to (81.3, 91.4)
- moved C8 89.2 mm to (88.9, 91.4)
- moved D2 89.0 mm to (101.6, 88.9)
- moved C5 79.1 mm to (91.4, 81.3), turned to 0 degrees
- moved R10 79.1 mm to (83.8, 76.2)
- moved C7 79.1 mm to (86.4, 86.4)
- moved SW1 75.8 mm to (109.2, 91.4)
- moved R4 75.2 mm to (121.9, 81.3)
- moved D3 65.9 mm to (127.0, 86.4)
- moved R4 34.1 mm to (119.4, 61.0)
- moved U1 34.1 mm to (101.6, 63.5)
- moved C11 34.1 mm to (76.2, 61.0)
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Connections:
- J1Power1 pad 1: +9V -> Net-(D8-Pad1)
Routing:
- net Net-(J2Signal1-Pad3): track 91.4 -> 10.2 mm, vias 0 -> 2
- net GND: track 226.0 -> 172.1 mm
- net +9V: track 129.5 -> 101.6 mm, vias 6 -> 9
- net Net-(C3-Pad2): track 61.0 -> 81.3 mm, vias 4 -> 6
- net Net-(RV1-Pad2): track 33.0 -> 12.7 mm
- net Net-(C3-Pad1): track 76.3 -> 58.5 mm, vias 2 -> 4
- net Net-(D1-Pad2): track 27.9 -> 12.7 mm, vias 2 -> 0
- net Net-(D3-Pad1): track 5.11 -> 14.6 mm
- net Net-(D3-Pad3): track 5.08 -> 14.6 mm
- net Net-(D8-Pad1): track 0.00 -> 5.08 mm
- net Net-(D3-Pad2): track 7.62 -> 5.08 mm, vias 2 -> 0
- net Net-(C8-Pad1): track 10.2 -> 12.7 mm
- net Net-(C7-Pad1): track 7.62 -> 10.2 mm
- net Net-(R3-Pad2): vias 5 -> 4
Other:
- board text added: "1"
- board text added: "10"
- board text added: "15"
- board text added: "18"
- board text added: "5"
- board text added: "A"
- board text added: "E"
- board text added: "J"
- board text added: "O"
- board text added: "T"
- board text added: "X"
